File: hardware/shifty.sch (EAGLE design)
At the start: 19 parts, among them IC1 74HC595D, IC2 74HC595D, IC3 ULN2003AD, IC4 ULN2003AD

Commit message: started routing
Parts:
- removed C1, C4, C5: (no value), rcl:C-EUC0805
- removed U$8: 2JUNCTION, shorts:2JUNCTION
Connections:
- removed net N$36 (its old number): IC4.O7, JP2.8
- new net +10V: IC3.CD+, IC4.CD+, JP1.2, JP1.4, JP1.6, JP2.2, JP2.4, JP2.6
- new net N$35: IC4.O4, JP2.8
- net GND: now also R1.1, R2.2; no longer U$8.P$1
- net GNDIO: no longer C1.2, C4.2, C5.2, R1.1, R2.2, U$8.P$2
- net N$10: now also IC2A.QC, IC4.I7; no longer IC2A.QB, IC4.I2
- net N$11: now also IC2A.QH, IC4.I2; no longer IC2A.QC, IC4.I3
- net N$12: now also IC4.I6; no longer IC4.I4
- net N$14: now also IC4.I4; no longer IC4.I6
- net N$15: now also IC4.I3; no longer IC4.I7
- net N$17: now also IC2A.QB; no longer IC2A.QH
- net N$2: now also IC1A.QH; no longer IC1A.QB
- net N$24: now also IC3.O5; no longer IC3.O4
- net N$25: now also IC3.O7; no longer IC3.O5
- net N$27: now also IC3.O4; no longer IC3.O7
- net N$3: now also IC3.I7; no longer IC3.I3
- net N$33: now also IC4.O5; no longer IC4.O4
- net N$34: now also IC4.O7; no longer IC4.O5
- net N$38: now also IC1A.QB; no longer IC1A.QH
- net N$4: now also IC3.I6; no longer IC3.I4
- net N$6: now also IC3.I4; no longer IC3.I6
- net N$7: now also IC3.I3; no longer IC3.I7
- net VCC: no longer C1.1, C4.1, C5.1, IC3.CD+, IC4.CD+, JP1.2, JP1.4, JP1.6, JP2.2, JP2.4, JP2.6

Commit message: Board lay-out done
Parts:
- removed JP3: (no value), pinhead:PINHD-1X4
- added JP10, JP6, JP7, JP8, JP9: (no value), adafruit:PINHD-1X1
Connections:
- net N$1: now also IC1A.QB; no longer IC1A.QA
- net N$16: now also JP6.1; no longer JP3.4
- net N$17: now also IC2A.QA; no longer IC2A.QB
- net N$18: now also JP10.1
- net N$20: now also JP9.1; no longer JP3.1
- net N$38: now also IC1A.QA; no longer IC1A.QB
- net N$43: now also JP7.1; no longer JP3.3
- net N$8: now also JP8.1; no longer JP3.2
- net N$9: now also IC2A.QB; no longer IC2A.QA
