File: hardware/shifty.brd (EAGLE design)
At the start: 35.2 x 43.2 mm, 19 parts, among them IC1 74HC595D, IC2 74HC595D, IC3 ULN2003AD, IC4 ULN2003AD

Commit message: started routing
Parts:
- removed C1, C4, C5: (no value), rcl:C0805
- removed U$8: 2JUNCTION, shorts:2JUNCTION
- moved C3 26.1 mm to (4.45, 28.2)
- moved LED2 15.7 mm to (31.8, 16.5)
- moved R2 11.6 mm to (32.4, 20.3)
- moved JP2 10.6 mm to (12.4, 5.61), turned to 180 degrees
- moved LED1 8.98 mm to (2.54, 21.6)
- moved IC1 4.47 mm to (25.4, 16.4)
- moved IC4 4.10 mm to (12.2, 16.3)
- moved R1 3.78 mm to (2.54, 28.2)
- moved IC3 2.74 mm to (25.4, 26.4)
- moved C2 2.69 mm to (32.4, 10.8)
- moved IC2 2.39 mm to (12.3, 26.4)
Connections:
- removed net N$36 (its old number): IC4.10, JP2.8
- new net +10V: IC3.9, IC4.9, JP1.2, JP1.4, JP1.6, JP2.2, JP2.4, JP2.6
- new net N$35: IC4.13, JP2.8
- net GND: now also R1.1, R2.2; no longer U$8.P$1
- net GNDIO: no longer C1.2, C4.2, C5.2, R1.1, R2.2, U$8.P$2
- net N$10: now also IC2.2, IC4.7; no longer IC2.1, IC4.2
- net N$11: now also IC2.7, IC4.2; no longer IC2.2, IC4.3
- net N$12: now also IC4.6; no longer IC4.4
- net N$14: now also IC4.4; no longer IC4.6
- net N$15: now also IC4.3; no longer IC4.7
- net N$17: now also IC2.1; no longer IC2.7
- net N$2: now also IC1.7; no longer IC1.1
- net N$24: now also IC3.12; no longer IC3.13
- net N$25: now also IC3.10; no longer IC3.12
- net N$27: now also IC3.13; no longer IC3.10
- net N$3: now also IC3.7; no longer IC3.3
- net N$33: now also IC4.12; no longer IC4.13
- net N$34: now also IC4.10; no longer IC4.12
- net N$38: now also IC1.1; no longer IC1.7
- net N$4: now also IC3.6; no longer IC3.4
- net N$6: now also IC3.4; no longer IC3.6
- net N$7: now also IC3.3; no longer IC3.7
- net VCC: no longer C1.1, C4.1, C5.1, IC3.9, IC4.9, JP1.2, JP1.4, JP1.6, JP2.2, JP2.4, JP2.6
Routing:
- net +10V: track 0.00 -> 44.8 mm
- net VCC: track 0.00 -> 18.2 mm
- net N$36: track 0.00 -> 10.0 mm
- net N$35: track 0.00 -> 10.0 mm
- net N$26: track 0.00 -> 9.80 mm
- net N$27: track 0.00 -> 9.40 mm
- net N$31: track 0.00 -> 7.71 mm
- net N$21: track 0.00 -> 7.38 mm
- net N$34: track 0.00 -> 6.98 mm
- net N$33: track 0.00 -> 6.98 mm
- net N$32: track 0.00 -> 6.98 mm
- net N$30: track 0.00 -> 6.67 mm
- net N$17: track 0.00 -> 6.50 mm
- net N$24: track 0.00 -> 6.44 mm
- net N$25: track 0.00 -> 6.33 mm
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- added copper zone on layer 16, net GND

Commit message: Board lay-out done
Parts:
- removed JP3: (no value), pinhead:1X04
- added JP10, JP6, JP7, JP8, JP9: (no value), adafruit:1X01
- moved JP1 29.3 mm to (24.8, 7.49), turned to 180 degrees
- moved C2 27.4 mm to (17.0, 33.5)
- moved LED2 21.3 mm to (18.5, 33.3)
- moved R2 18.0 mm to (20.1, 33.4), turned to 270 degrees
- moved LED1 13.5 mm to (9.27, 33.3)
- moved IC3 10.4 mm to (23.1, 16.3), turned to 180 degrees
- moved IC1 10.0 mm to (23.2, 26.2), turned to 0 degrees
- moved R1 9.69 mm to (10.8, 33.3), turned to 90 degrees
- moved JP5 8.63 mm to (21.7, 38.1)
- moved C3 6.27 mm to (7.75, 33.5)
- moved JP4 2.67 mm to (7.75, 38.1), turned to 180 degrees
- moved JP2 2.16 mm to (11.4, 7.52)
- moved IC2 0.28 mm to (12.2, 26.2)
Connections:
- net N$1: now also IC1.1; no longer IC1.15
- net N$16: now also JP6.1; no longer JP3.4
- net N$17: now also IC2.15; no longer IC2.1
- net N$18: now also JP10.1
- net N$20: now also JP9.1; no longer JP3.1
- net N$38: now also IC1.15; no longer IC1.1
- net N$43: now also JP7.1; no longer JP3.3
- net N$8: now also JP8.1; no longer JP3.2
- net N$9: now also IC2.1; no longer IC2.15
Routing:
- net GND: track 0.00 -> 66.9 mm, vias 0 -> 5
- net N$18: track 0.00 -> 39.0 mm
- net N$20: track 0.00 -> 31.7 mm, vias 0 -> 2
- net N$8: track 0.00 -> 27.7 mm
- net N$43: track 0.00 -> 27.6 mm
- net N$19: track 0.00 -> 24.4 mm
- net N$1: track 0.00 -> 19.0 mm
- net N$9: track 0.00 -> 16.0 mm
- net GNDIO: track 0.00 -> 15.2 mm, vias 0 -> 2
- net N$29: track 0.00 -> 12.8 mm, vias 0 -> 3
- net N$16: track 0.00 -> 11.3 mm, vias 0 -> 1
- net VCC: track 18.2 -> 27.2 mm, vias 0 -> 2
- net N$28: track 5.34 -> 1.53 mm
- net +10V: track 44.8 -> 48.5 mm
- net N$17: track 6.50 -> 3.30 mm
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- added copper zone on layer 16, net N$39
- removed copper zone on layer 16, net GND
Other:
- board size 35.2 x 43.2 mm -> 28.6 x 38.5 mm

Commit message: Board lay-out done
Other:
- board size 28.6 x 38.5 mm -> 27.9 x 36.6 mm
